Commit message: Add files via upload

File: urdf/fckwv1.xacro (robot description, xacro)
@@ -1,7 +1,4 @@
 <?xml version="1.0" ?>
 <robot name="fckwv1" xmlns:xacro="http://www.ros.org/wiki/xacro">
-<xacro:include filename="$(find fckwv1_description)/urdf/materials.xacro" />
-<xacro:include filename="$(find fckwv1_description)/urdf/fckwv1.trans" />
-<xacro:include filename="$(find fckwv1_description)/urdf/diff_drive.gazebo" />
 <link name="base_link">
   <inertial>
@@ -25,4 +22,6 @@
 </link>
 <link name="base_footprint">
+</link>
+<link name="laser_frame">
 </link>
 <link name="rear_wheel_link_1_1">
@@ -106,5 +105,5 @@
   </collision>
 </link>
-<link name="laser_frame">
+<link name="lidar_link">
   <inertial>
     <origin xyz="-4.4699088558586286e-05 1.0188628332296945e-07 0.020292487366021572" rpy="0 0 0"/>
@@ -173,4 +172,9 @@
   <origin xyz="0.195004 0.0 0.346999" rpy="0 0 0"/>
   <parent link="base_link"/>
+  <child link="lidar_link"/>
+</joint>
+<joint name="lidar_scan" type="fixed">
+  <origin xyz="0.0 0.0 0.042" rpy="0 0 0"/>
+  <parent link="lidar_link"/>
   <child link="laser_frame"/>
 </joint>
